File: hardware/_autosave-hardware.kicad_pcb (KiCad board)
At the start: 2 copper layers, 56 parts, among them J101 VIN, J102 BAT, J103 DISPLAY, J104 EXT, J105 VIN, J106 SENSOR_DHT, J107 solo, SW101 BOOT, U101 LM324, U102 TP4056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

Commit message: pcb
Parts:
- moved C104 80.9 mm to (117.4, 149.5)
- moved U103 6.60 mm to (122.6, 143.7)
Changed lines of the file:
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@@
   )
   (footprint "Package_TO_SOT_SMD:SOT-23-6_Handsoldering" (layer "B.Cu")
-    (at 121.5975 150.2 180)
+    (at 122.6375 143.68 180)
     (descr "6-pin SOT-23 package, Handsoldering")
     (tags "SOT-23-6 Handsoldering")
@@
   )
   (footprint "Capacitor_SMD:C_0805_2012Metric_Pad1.18x1.45mm_HandSolder" (layer "B.Cu")
-    (at 56.3375 96.47 180)
+    (at 117.4475 149.47 180)
     (descr "Capacitor SMD 0805 (2012 Metric), square (rectangular) end terminal, IPC_7351 nominal with elongated pad for handsoldering. (Body size source: IPC-SM-782 page 76, https://www.pcb-3d.com/wordpress/wp-content/uploads/ipc-sm-782a_amendment_1_and_2.pdf, https://docs.google.com/spreadsheets/d/1BsfQQcO9C6DZCsRaXUlFlo91Tg2WpOkGARC1WS5S8t0/edit?usp=sharing), generated with kicad-footprint-generator")
     (tags "capacitor handsolder")
