File: hardware/hardware.kicad_pcb (KiCad board)
At the start: 2 copper layers, 56 parts, among them J101 VIN, J102 BAT, J103 DISPLAY, J104 EXT, J105 VIN, J106 SENSOR_DHT, J107 solo, SW101 BOOT, U101 LM324, U102 TP4056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

Commit message: pcb
Parts:
- moved R109 126.6 mm to (165.1, 145.0)
- moved R117 108.5 mm to (169.2, 175.6)
- moved J101 105.9 mm to (150.1, 176.6)
- moved R110 105.9 mm to (164.5, 188.9)
- moved R111 105.9 mm to (145.3, 191.2)
- moved R116 105.9 mm to (159.7, 192.0)
- moved C111 105.9 mm to (161.4, 163.3)
- moved D103 105.9 mm to (159.6, 186.0)
- moved D104 105.9 mm to (162.4, 169.3)
- moved D105 105.9 mm to (154.9, 175.5)
- moved D106 105.9 mm to (148.8, 184.4)
- moved R115 100.0 mm to (151.0, 135.9)
- moved R114 97.8 mm to (157.3, 140.2)
- moved R112 89.8 mm to (147.6, 131.2)
- moved C104 77.6 mm to (117.2, 144.6)
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Routing:
- net Net-(C113-Pad2): track 0.00 -> 7.06 mm
- net /IO0: track 5.14 -> 12.0 mm
- net /VBAT: track 0.00 -> 6.63 mm
- net GND: track 15.0 -> 20.2 mm
- net Net-(R108-Pad1): track 4.85 -> 0.00 mm
- net Net-(C103-Pad1): track 8.03 -> 12.8 mm
- net Net-(C101-Pad1): track 14.4 -> 9.74 mm
- net /ADC_EXT: track 7.30 -> 3.85 mm
- net BAT+: track 0.00 -> 2.45 mm
- net Net-(R120-Pad1): track 0.00 -> 1.27 mm
- net Net-(R119-Pad1): track 0.00 -> 1.27 mm
- net /SENS_SOLO: track 0.00 -> 1.27 mm
- net /LUMINOSIDADE: track 0.00 -> 1.27 mm

Commit message: Update hardware.kicad_pcb
Parts:
- moved J103 32.1 mm to (99.0, 109.7)
- moved J102 23.8 mm to (98.0, 150.0)
- moved C104 21.4 mm to (97.0, 137.5), turned to -90 degrees
- moved C110 11.5 mm to (117.5, 149.2)
- moved R102 3.66 mm to (117.0, 138.4)
- moved R108 2.58 mm to (120.1, 132.1)
Routing:
- net BAT+: track 2.45 -> 30.9 mm
- net Net-(R108-Pad1): track 0.00 -> 7.02 mm
Changed lines of the file:
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@@
   (net 66 "unconnected-(U107-Pad3)")
   (footprint "Connector_PinHeader_2.54mm:PinHeader_1x02_P2.54mm_Vertical" (layer "F.Cu")
-    (at 76.1575 140.555)
+    (at 98.0275 149.97)
     (descr "Through hole straight pin header, 1x02, 2.54mm pitch, single row")
     (tags "Through hole pin header THT 1x02 2.54mm single row")
@@
       (effects (font (size 1 1) (thickness 0.15)))
     )
-    (fp_text user "${REFERENCE}" (at 0.31 5.205 180) (layer "F.Fab")
+    (fp_text user "${REFERENCE}" (at 0.31 5.205) (layer "F.Fab")
       (effects (font (size 1 1) (thickness 0.15)))
     )
@@
   )
   (footprint "Connector_PinSocket_2.54mm:PinSocket_1x04_P2.54mm_Vertical" (layer "F.Cu")
-    (at 76.9975 133.02 180)
+    (at 99.0425 109.74 180)
     (descr "Through hole straight socket strip, 1x04, 2.54mm pitch, single row (from Kicad 4.0.7), script generated")
     (tags "Through hole socket strip THT 1x04 2.54mm single row")
@@
   )
   (footprint "Resistor_SMD:R_0805_2012Metric_Pad1.20x1.40mm_HandSolder" (layer "B.Cu")
-    (at 117.5475 132.43)
+    (at 120.1075 132.11)
     (descr "Resistor SMD 0805 (2012 Metric), square (rectangular) end terminal, IPC_7351 nominal with elongated pad for handsoldering. (Body size source: IPC-SM-782 page 72, https://www.pcb-3d.com/wordpress/wp-content/uploads/ipc-sm-782a_amendment_1_and_2.pdf), generated with kicad-footprint-generator")
     (tags "resistor handsolder")
@@
   )
   (footprint "Resistor_SMD:R_0805_2012Metric_Pad1.20x1.40mm_HandSolder" (layer "B.Cu")
-    (at 119.6125 135.805)
+    (at 117.0475 138.42)
     (descr "Resistor SMD 0805 (2012 Metric), square (rectangular) end terminal, IPC_7351 nominal with elongated pad for handsoldering. (Body size source: IPC-SM-782 page 72, https://www.pcb-3d.com/wordpress/wp-content/uploads/ipc-sm-782a_amendment_1_and_2.pdf), generated with kicad-footprint-generator")
     (tags "resistor handsolder")
@@
   )
   (footprint "Capacitor_SMD:C_0805_2012Metric_Pad1.18x1.45mm_HandSolder" (layer "B.Cu")
-    (at 117.19 144.55 180)
+    (at 96.9875 137.48 -90)
     (descr "Capacitor SMD 0805 (2012 Metric), square (rectangular) end terminal, IPC_7351 nominal with elongated pad for handsoldering. (Body size source: IPC-SM-782 page 76, https://www.pcb-3d.com/wordpress/wp-content/uploads/ipc-sm-782a_amendment_1_and_2.pdf, https://docs.google.com/spreadsheets/d/1BsfQQcO9C6DZCsRaXUlFlo91Tg2WpOkGARC1WS5S8t0/edit?usp=sharing), generated with kicad-footprint-generator")
     (tags "capacitor handsolder")
@@
     (property "Sheetname" "")
     (attr smd)
-    (fp_text reference "C104" (at 0 1.68) (layer "B.SilkS")
-      (effects (font (size 1 1) (thickness 0.15)) (justify mirror))
-    )
-    (fp_text value "100nF" (at 0 -1.68) (layer "B.Fab")
-      (effects (font (size 1 1) (thickness 0.15)) (justify mirror))
-    )
-    (fp_text user "${REFERENCE}" (at 0 0) (layer "B.Fab")
+    (fp_text reference "C104" (at 2.78 -0.34) (layer "B.SilkS")
+      (effects (font (size 1 1) (thickness 0.15)) (justify mirror))
+    )
+    (fp_text value "100nF" (at -0.31 -1.84 90) (layer "B.Fab")
+      (effects (font (size 1 1) (thickness 0.15)) (justify mirror))
+    )
+    (fp_text user "${REFERENCE}" (at 0 0 90) (layer "B.Fab")
       (effects (font (size 0.5 0.5) (thickness 0.08)) (justify mirror))
     )
@@
     (fp_line (start -1 0.625) (end 1 0.625) (layer "B.Fab") (width 0.1))
     (fp_line (start -1 -0.625) (end -1 0.625) (layer "B.Fab") (width 0.1))
-    (pad "1" smd roundrect (at -1.0375 0 180) (size 1.175 1.45) (layers "B.Cu" "B.Paste" "B.Mask") (roundrect_rratio 0.212766)
+    (pad "1" smd roundrect (at -1.0375 0 270) (size 1.175 1.45) (layers "B.Cu" "B.Paste" "B.Mask") (roundrect_rratio 0.212766)
       (net 6 "BAT+") (pintype "passive"))
-    (pad "2" smd roundrect (at 1.0375 0 180) (size 1.175 1.45) (layers "B.Cu" "B.Paste" "B.Mask") (roundrect_rratio 0.212766)
+    (pad "2" smd roundrect (at 1.0375 0 270) (size 1.175 1.45) (layers "B.Cu" "B.Paste" "B.Mask") (roundrect_rratio 0.212766)
       (net 4 "GND") (pintype "passive"))
     (model "${KICAD6_3DMODEL_DIR}/Capacitor_SMD.3dshapes/C_0805_2012Metric.wrl"
@@
   )
   (footprint "Capacitor_SMD:C_0805_2012Metric_Pad1.18x1.45mm_HandSolder" (layer "B.Cu")
-    (at 114.26 160.26 180)
+    (at 117.54 149.19 180)
     (descr "Capacitor SMD 0805 (2012 Metric), square (rectangular) end terminal, IPC_7351 nominal with elongated pad for handsoldering. (Body size source: IPC-SM-782 page 76, https://www.pcb-3d.com/wordpress/wp-content/uploads/ipc-sm-782a_amendment_1_and_2.pdf, https://docs.google.com/spreadsheets/d/1BsfQQcO9C6DZCsRaXUlFlo91Tg2WpOkGARC1WS5S8t0/edit?usp=sharing), generated with kicad-footprint-generator")
     (tags "capacitor handsolder")
@@
   (segment (start 112.1175 140.92) (end 112.2875 141.09) (width 0.25) (layer "B.Cu") (net 5))
   (segment (start 112.2875 141.46) (end 112.1775 141.35) (width 0.25) (layer "B.Cu") (net 5))
+  (segment (start 98.0275 141) (end 98.7475 140.28) (width 0.25) (layer "B.Cu") (net 6))
+  (segment (start 108.5675 132.07) (end 108.5675 131.61) (width 0.25) (layer "B.Cu") (net 6))
   (segment (start 110.9975 131.55) (end 108.6275 131.55) (width 0.25) (layer "B.Cu") (net 6))
+  (segment (start 99.67 133.76) (end 106.8775 133.76) (width 0.25) (layer "B.Cu") (net 6))
+  (segment (start 98.7475 140.28) (end 98.7475 138.15) (width 0.25) (layer "B.Cu") (net 6))
+  (segment (start 96.9875 136.4425) (end 99.67 133.76) (width 0.25) (layer "B.Cu") (net 6))
+  (segment (start 97.04 136.4425) (end 96.9875 136.4425) (width 0.25) (layer "B.Cu") (net 6))
+  (segment (start 106.8775 133.76) (end 108.5675 132.07) (width 0.25) (layer "B.Cu") (net 6))
+  (segment (start 98.7475 138.15) (end 97.04 136.4425) (width 0.25) (layer "B.Cu") (net 6))
   (segment (start 108.6275 131.55) (end 108.5675 131.61) (width 0.25) (layer "B.Cu") (net 6))
+  (segment (start 98.0275 149.97) (end 98.0275 141) (width 0.25) (layer "B.Cu") (net 6))
   (segment (start 132.0775 113.695) (end 131.9125 113.53) (width 0.25) (layer "B.Cu") (net 7))
   (segment (start 131.9125 113.53) (end 129.0275 113.53) (width 0.25) (layer "B.Cu") (net 7))
@@
   (segment (start 109.1775 119.98) (end 109.1775 117.73) (width 0.25) (layer "B.Cu") (net 19))
   (segment (start 109.1775 119.98) (end 109.3425 119.815) (width 0.25) (layer "B.Cu") (net 19))
+  (segment (start 116.3275 132.11) (end 119.1075 132.11) (width 0.25) (layer "B.Cu") (net 20))
+  (segment (start 114.8125 130.595) (end 116.3275 132.11) (width 0.25) (layer "B.Cu") (net 20))
+  (segment (start 114.8125 128.5) (end 114.8125 130.595) (width 0.25) (layer "B.Cu") (net 20))
   (segment (start 132.185 117.285) (end 132.13 117.34) (width 0.25) (layer "B.Cu") (net 25))
   (segment (start 132.13 117.34) (end 129.0275 117.34) (width 0.25) (layer "B.Cu") (net 25))

Commit message: esq e pcb
Parts:
- moved D105 57.4 mm to (172.1, 120.7)
- moved D103 57.4 mm to (176.9, 131.3)
- moved D104 57.4 mm to (179.6, 114.6)
- moved R110 57.4 mm to (181.8, 134.2)
- moved R117 57.4 mm to (186.5, 120.9)
- moved D106 57.4 mm to (166.1, 129.7)
- moved J101 57.4 mm to (167.4, 121.8)
- moved R111 57.4 mm to (162.6, 136.5)
- moved R116 57.4 mm to (177.0, 137.2)
- moved C111 55.2 mm to (139.3, 112.7), turned to 90 degrees
- moved C110 11.8 mm to (123.1, 138.8)
- moved D102 10.3 mm to (110.4, 152.9)
- moved D101 6.05 mm to (124.6, 154.1)
- moved U101 3.54 mm to (139.4, 130.9)
- moved R121 2.04 mm to (133.6, 123.4)
Connections:
- U106 pad 33: unconnected-(U106-Pad33) -> /SDA
- U106 pad 36: unconnected-(U106-Pad36) -> /SCL
Routing:
- net Net-(D102-Pad2): track 9.74 -> 36.8 mm
- net +3V3: track 15.5 -> 24.0 mm
- net Net-(C113-Pad2): track 7.06 -> 0.00 mm
- net GND: track 20.2 -> 24.7 mm
- net Net-(D101-Pad1): track 5.27 -> 0.74 mm
- net /ADC_EXT: track 3.85 -> 0.00 mm
- net Net-(R120-Pad1): track 1.27 -> 0.00 mm
- net Net-(R119-Pad1): track 1.27 -> 0.00 mm
- net /SENS_SOLO: track 1.27 -> 0.00 mm
- net /LUMINOSIDADE: track 1.27 -> 0.00 mm

Commit message: Update hardware.kicad_pcb
Parts:
- moved R107 3.46 mm to (108.4, 123.4), turned to -90 degrees
- moved R113 2.30 mm to (106.6, 119.4)
- moved C109 1.54 mm to (98.9, 120.1)
- moved SW101 1.54 mm to (102.3, 120.3)
- moved J103 1.09 mm to (98.0, 109.5)
Routing:
- net +3V3: track 24.0 -> 43.6 mm
- net /SDA: track 0.00 -> 18.4 mm
- net /SCL: track 0.00 -> 17.8 mm
- net GND: track 24.7 -> 42.5 mm
- net Net-(C109-Pad2): track 10.3 -> 9.04 mm
- net /IO0: track 12.0 -> 12.5 mm

Commit message: Update hardware.kicad_pcb
Parts:
- moved R117 65.7 mm to (121.9, 132.7)
- moved R108 3.23 mm to (116.9, 132.7)
- moved C104 2.82 mm to (98.6, 135.2), turned to 90 degrees
Routing:
- net GND: track 42.5 -> 90.8 mm
- net /STDB: track 0.00 -> 5.06 mm
- net BAT+: track 30.9 -> 28.3 mm
- net Net-(R108-Pad1): track 7.02 -> 4.66 mm
Changed lines of the file:
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@@
     (property "Sheetname" "")
     (attr smd)
-    (fp_text reference "R106" (at 0.0175 -1.61) (layer "B.SilkS")
+    (fp_text reference "R106" (at -0.0125 1.6) (layer "B.SilkS")
       (effects (font (size 1 1) (thickness 0.15)) (justify mirror))
     )
@@
   )
   (footprint "Resistor_SMD:R_0805_2012Metric_Pad1.20x1.40mm_HandSolder" (layer "B.Cu")
-    (at 120.1075 132.11)
+    (at 116.9275 132.7)
     (descr "Resistor SMD 0805 (2012 Metric), square (rectangular) end terminal, IPC_7351 nominal with elongated pad for handsoldering. (Body size source: IPC-SM-782 page 72, https://www.pcb-3d.com/wordpress/wp-content/uploads/ipc-sm-782a_amendment_1_and_2.pdf), generated with kicad-footprint-generator")
     (tags "resistor handsolder")
@@
     (property "Sheetname" "")
     (attr smd)
-    (fp_text reference "C106" (at 2.81 -0.42 90) (layer "B.SilkS")
+    (fp_text reference "C106" (at 0.08 1.6 180) (layer "B.SilkS")
       (effects (font (size 1 1) (thickness 0.15)) (justify mirror))
     )
@@
       (effects (font (size 1 1) (thickness 0.15)) (justify mirror))
     )
-    (fp_text value "R" (at 1.16 1.73 180) (layer "B.Fab")
+    (fp_text value "R" (at -0.04 1.6 180) (layer "B.Fab")
       (effects (font (size 1 1) (thickness 0.15)) (justify mirror))
     )
@@
   )
   (footprint "Resistor_SMD:R_0805_2012Metric_Pad1.20x1.40mm_HandSolder" (layer "B.Cu")
-    (at 186.515 120.865 180)
+    (at 121.9075 132.7 180)
     (descr "Resistor SMD 0805 (2012 Metric), square (rectangular) end terminal, IPC_7351 nominal with elongated pad for handsoldering. (Body size source: IPC-SM-782 page 72, https://www.pcb-3d.com/wordpress/wp-content/uploads/ipc-sm-782a_amendment_1_and_2.pdf), generated with kicad-footprint-generator")
     (tags "resistor handsolder")
@@
     (property "Sheetname" "")
     (attr smd)
-    (fp_text reference "R117" (at 0 1.65) (layer "B.SilkS")
+    (fp_text reference "R117" (at 0.03 -1.79) (layer "B.SilkS")
       (effects (font (size 1 1) (thickness 0.15)) (justify mirror))
     )
@@
   )
   (footprint "Capacitor_SMD:C_0805_2012Metric_Pad1.18x1.45mm_HandSolder" (layer "B.Cu")
-    (at 96.9875 137.48 -90)
+    (at 98.5975 135.1625 90)
     (descr "Capacitor SMD 0805 (2012 Metric), square (rectangular) end terminal, IPC_7351 nominal with elongated pad for handsoldering. (Body size source: IPC-SM-782 page 76, https://www.pcb-3d.com/wordpress/wp-content/uploads/ipc-sm-782a_amendment_1_and_2.pdf, https://docs.google.com/spreadsheets/d/1BsfQQcO9C6DZCsRaXUlFlo91Tg2WpOkGARC1WS5S8t0/edit?usp=sharing), generated with kicad-footprint-generator")
     (tags "capacitor handsolder")
@@
     (property "Sheetname" "")
     (attr smd)
-    (fp_text reference "C104" (at 2.78 -0.34) (layer "B.SilkS")
-      (effects (font (size 1 1) (thickness 0.15)) (justify mirror))
-    )
-    (fp_text value "100nF" (at -0.31 -1.84 90) (layer "B.Fab")
+    (fp_text reference "C104" (at -2.6875 -0.86 180) (layer "B.SilkS")
+      (effects (font (size 1 1) (thickness 0.15)) (justify mirror))
+    )
+    (fp_text value "100nF" (at 0.63 -1.69 270) (layer "B.Fab")
       (effects (font (size 1 1) (thickness 0.15)) (justify mirror))
     )
@@
     (fp_line (start -1 0.625) (end 1 0.625) (layer "B.Fab") (width 0.1))
     (fp_line (start -1 -0.625) (end -1 0.625) (layer "B.Fab") (width 0.1))
-    (pad "1" smd roundrect (at -1.0375 0 270) (size 1.175 1.45) (layers "B.Cu" "B.Paste" "B.Mask") (roundrect_rratio 0.212766)
+    (pad "1" smd roundrect (at -1.0375 0 90) (size 1.175 1.45) (layers "B.Cu" "B.Paste" "B.Mask") (roundrect_rratio 0.212766)
       (net 6 "BAT+") (pintype "passive"))
-    (pad "2" smd roundrect (at 1.0375 0 270) (size 1.175 1.45) (layers "B.Cu" "B.Paste" "B.Mask") (roundrect_rratio 0.212766)
+    (pad "2" smd roundrect (at 1.0375 0 90) (size 1.175 1.45) (layers "B.Cu" "B.Paste" "B.Mask") (roundrect_rratio 0.212766)
       (net 4 "GND") (pintype "passive"))
     (model "${KICAD6_3DMODEL_DIR}/Capacitor_SMD.3dshapes/C_0805_2012Metric.wrl"
@@
   (segment (start 147.7925 148.53) (end 146.1625 146.9) (width 0.25) (layer "B.Cu") (net 4))
   (segment (start 98.8975 121.1275) (end 99.225 121.1275) (width 0.25) (layer "B.Cu") (net 4))
+  (segment (start 96.5775 151.06) (end 96.5775 136.01) (width 0.25) (layer "B.Cu") (net 4))
+  (segment (start 98.5975 134.125) (end 99.115 134.125) (width 0.25) (layer "B.Cu") (net 4))
+  (segment (start 96.5775 136.01) (end 98.4625 134.125) (width 0.25) (layer "B.Cu") (net 4))
   (segment (start 102.3275 124.23) (end 102.3275 127.1875) (width 0.25) (layer "B.Cu") (net 4))
   (segment (start 99.225 121.1275) (end 102.3275 124.23) (width 0.25) (layer "B.Cu") (net 4))
   (segment (start 97.9925 101.83) (end 99.4975 101.83) (width 0.25) (layer "B.Cu") (net 4))
+  (segment (start 97.9925 101.83) (end 96.0075 103.815) (width 0.25) (layer "B.Cu") (net 4))
   (segment (start 139.3075 113.735) (end 138.7825 113.735) (width 0.25) (layer "B.Cu") (net 4))
+  (segment (start 96.0075 118.2375) (end 98.8975 121.1275) (width 0.25) (layer "B.Cu") (net 4))
   (segment (start 101.63 127.935) (end 101.605 127.91) (width 0.25) (layer "B.Cu") (net 4))
+  (segment (start 98.0275 152.51) (end 96.5775 151.06) (width 0.25) (layer "B.Cu") (net 4))
+  (segment (start 117.9275 132.7) (end 120.9075 132.7) (width 0.25) (layer "B.Cu") (net 4))
+  (segment (start 98.4625 134.125) (end 98.5975 134.125) (width 0.25) (layer "B.Cu") (net 4))
   (segment (start 138.7825 113.735) (end 136.645 111.5975) (width 0.25) (layer "B.Cu") (net 4))
+  (segment (start 96.0075 103.815) (end 96.0075 118.2375) (width 0.25) (layer "B.Cu") (net 4))
   (segment (start 100.3675 105.34) (end 106.0175 110.99) (width 0.25) (layer "B.Cu") (net 4))
   (segment (start 106.0175 110.99) (end 112.0275 110.99) (width 0.25) (layer "B.Cu") (net 4))
@@
   (segment (start 102.3275 127.1875) (end 101.605 127.91) (width 0.25) (layer "B.Cu") (net 4))
   (segment (start 136.645 111.5975) (end 135.6475 111.5975) (width 0.25) (layer "B.Cu") (net 4))
+  (segment (start 99.115 134.125) (end 101.63 131.61) (width 0.25) (layer "B.Cu") (net 4))
   (segment (start 99.4975 101.83) (end 100.3675 102.7) (width 0.25) (layer "B.Cu") (net 4))
   (segment (start 147.7925 152.38) (end 147.7925 148.53) (width 0.25) (layer "B.Cu") (net 4))
@@
   (segment (start 112.1175 140.92) (end 112.2875 141.09) (width 0.25) (layer "B.Cu") (net 5))
   (segment (start 112.2875 141.46) (end 112.1775 141.35) (width 0.25) (layer "B.Cu") (net 5))
-  (segment (start 98.0275 141) (end 98.7475 140.28) (width 0.25) (layer "B.Cu") (net 6))
-  (segment (start 108.5675 132.07) (end 108.5675 131.61) (width 0.25) (layer "B.Cu") (net 6))
+  (segment (start 98.5975 136.2) (end 103.9775 136.2) (width 0.25) (layer "B.Cu") (net 6))
   (segment (start 110.9975 131.55) (end 108.6275 131.55) (width 0.25) (layer "B.Cu") (net 6))
-  (segment (start 99.67 133.76) (end 106.8775 133.76) (width 0.25) (layer "B.Cu") (net 6))
-  (segment (start 98.7475 140.28) (end 98.7475 138.15) (width 0.25) (layer "B.Cu") (net 6))
-  (segment (start 96.9875 136.4425) (end 99.67 133.76) (width 0.25) (layer "B.Cu") (net 6))
-  (segment (start 97.04 136.4425) (end 96.9875 136.4425) (width 0.25) (layer "B.Cu") (net 6))
-  (segment (start 106.8775 133.76) (end 108.5675 132.07) (width 0.25) (layer "B.Cu") (net 6))
-  (segment (start 98.7475 138.15) (end 97.04 136.4425) (width 0.25) (layer "B.Cu") (net 6))
+  (segment (start 103.9775 136.2) (end 108.5675 131.61) (width 0.25) (layer "B.Cu") (net 6))
   (segment (start 108.6275 131.55) (end 108.5675 131.61) (width 0.25) (layer "B.Cu") (net 6))
-  (segment (start 98.0275 149.97) (end 98.0275 141) (width 0.25) (layer "B.Cu") (net 6))
+  (segment (start 98.0275 149.97) (end 98.0275 136.77) (width 0.25) (layer "B.Cu") (net 6))
+  (segment (start 98.0275 136.77) (end 98.5975 136.2) (width 0.25) (layer "B.Cu") (net 6))
   (segment (start 132.0775 113.695) (end 131.9125 113.53) (width 0.25) (layer "B.Cu") (net 7))
   (segment (start 131.9125 113.53) (end 129.0275 113.53) (width 0.25) (layer "B.Cu") (net 7))
@@
   (segment (start 110.0375 127.5) (end 108.3975 125.86) (width 0.25) (layer "B.Cu") (net 19))
   (segment (start 112.0275 127.5) (end 110.0375 127.5) (width 0.25) (layer "B.Cu") (net 19))
-  (segment (start 116.3275 132.11) (end 119.1075 132.11) (width 0.25) (layer "B.Cu") (net 20))
-  (segment (start 114.8125 130.595) (end 116.3275 132.11) (width 0.25) (layer "B.Cu") (net 20))
-  (segment (start 114.8125 128.5) (end 114.8125 130.595) (width 0.25) (layer "B.Cu") (net 20))
+  (segment (start 114.8125 131.585) (end 114.8125 128.5) (width 0.25) (layer "B.Cu") (net 20))
+  (segment (start 115.9275 132.7) (end 114.8125 131.585) (width 0.25) (layer "B.Cu") (net 20))
   (segment (start 132.185 117.285) (end 132.13 117.34) (width 0.25) (layer "B.Cu") (net 25))
   (segment (start 132.13 117.34) (end 129.0275 117.34) (width 0.25) (layer "B.Cu") (net 25))
+  (segment (start 124.9725 130.635) (end 124.9725 128.5) (width 0.25) (layer "B.Cu") (net 30))
+  (segment (start 122.9075 132.7) (end 124.9725 130.635) (width 0.25) (layer "B.Cu") (net 30))
 )

Commit message: pcb update
Parts:
- C101, C103, C107, C108, C110, C113, D101, D102, R101, R122, U101, U102: moved to F.Cu
- moved J101 75.1 mm to (97.8, 150.2)
- moved J104 59.7 mm to (146.0, 112.2), turned to 180 degrees
- moved J106 53.2 mm to (169.8, 149.3)
- moved D104 44.2 mm to (151.9, 149.0)
- moved R110 44.2 mm to (138.9, 145.0)
- moved R116 43.2 mm to (137.0, 153.5)
- moved D103 42.1 mm to (134.8, 130.3), turned to 90 degrees
- moved C111 40.9 mm to (98.4, 113.0), turned to 0 degrees
- moved R109 34.0 mm to (132.5, 135.3)
- moved R114 29.9 mm to (127.9, 135.2)
- moved C108 27.7 mm to (122.2, 144.9), turned to 0 degrees
- moved C107 26.8 mm to (122.7, 139.4), turned to 0 degrees
- moved R111 26.7 mm to (139.8, 122.5)
- moved D105 26.4 mm to (145.9, 117.6), turned to 0 degrees
- moved R115 23.5 mm to (127.8, 131.8)
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Connections:
- U101 pad 8: /LUMINOSIDADE -> /LUX_ADC
- U101 pad 9: /LUMINOSIDADE -> /LUX_ADC
Routing:
- net Net-(J104-Pad2): track 0.00 -> 74.8 mm, vias 0 -> 1
- net BAT+: track 28.3 -> 64.6 mm, vias 0 -> 1
- net Net-(D101-Pad1): track 0.74 -> 34.0 mm, vias 0 -> 1
- net Net-(R120-Pad1): track 0.00 -> 31.9 mm, vias 0 -> 1
- net Net-(R119-Pad1): track 0.00 -> 28.6 mm, vias 0 -> 1
- net +3V3: track 43.6 -> 68.4 mm
- net /VBAT: track 6.63 -> 30.0 mm, vias 0 -> 1
- net GND: track 90.8 -> 108.2 mm
- net Net-(U103-Pad3): track 0.00 -> 17.4 mm
- net /DHT: track 0.00 -> 17.3 mm
- net GND1: track 7.15 -> 22.4 mm
- net /ADC_EXT: track 0.00 -> 14.2 mm
- net /CHG: track 0.00 -> 12.3 mm
- net /SENS_SOLO: track 0.00 -> 11.8 mm, vias 0 -> 1
- net /LUX_ADC: track 0.00 -> 11.5 mm, vias 0 -> 1
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