File: hardware/hardware.kicad_pcb (KiCad board)
At the start: 2 copper layers, 56 parts, among them J101 VIN, J102 BAT, J103 DISPLAY, J104 EXT, J105 VIN, J106 SENSOR_DHT, J107 solo, SW101 BOOT, U101 LM324, U102 TP4056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

Commit message: Update hardware.kicad_pcb
Parts:
- moved J106 32.5 mm to (145.9, 127.4), turned to 180 degrees
- moved U107 21.0 mm to (166.6, 129.4)
- moved R116 10.5 mm to (130.5, 145.3)
Routing:
- net GND: track 108.2 -> 121.4 mm
- net +3V3: track 68.4 -> 78.2 mm
- net /DHT: track 17.3 -> 18.7 mm
Changed lines of the file:
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@@
   )
   (footprint "Sensor:Aosong_DHT11_5.5x12.0_P2.54mm" (layer "F.Cu")
-    (at 145.54 129.4225 180)
+    (at 166.5875 129.43 180)
     (descr "Temperature and humidity module, http://akizukidenshi.com/download/ds/aosong/DHT11.pdf")
     (tags "Temperature and humidity module")
@@
   )
   (footprint "Connector_PinHeader_2.54mm:PinHeader_1x03_P2.54mm_Vertical" (layer "F.Cu")
-    (at 169.8175 149.265)
+    (at 145.8675 127.365 180)
     (descr "Through hole straight pin header, 1x03, 2.54mm pitch, single row")
     (tags "Through hole pin header THT 1x03 2.54mm single row")
@@
     (fp_line (start -0.635 -1.27) (end 1.27 -1.27) (layer "F.Fab") (width 0.1))
     (fp_line (start -1.27 6.35) (end -1.27 -0.635) (layer "F.Fab") (width 0.1))
-    (pad "1" thru_hole rect (at 0 0) (size 1.7 1.7) (drill 1) (layers *.Cu *.Mask)
+    (pad "1" thru_hole rect (at 0 0 180) (size 1.7 1.7) (drill 1) (layers *.Cu *.Mask)
       (net 3 "+3V3") (pinfunction "Pin_1") (pintype "passive"))
-    (pad "2" thru_hole oval (at 0 2.54) (size 1.7 1.7) (drill 1) (layers *.Cu *.Mask)
+    (pad "2" thru_hole oval (at 0 2.54 180) (size 1.7 1.7) (drill 1) (layers *.Cu *.Mask)
       (net 62 "/DHT") (pinfunction "Pin_2") (pintype "passive"))
-    (pad "3" thru_hole oval (at 0 5.08) (size 1.7 1.7) (drill 1) (layers *.Cu *.Mask)
+    (pad "3" thru_hole oval (at 0 5.08 180) (size 1.7 1.7) (drill 1) (layers *.Cu *.Mask)
       (net 4 "GND") (pinfunction "Pin_3") (pintype "passive"))
     (model "${KICAD6_3DMODEL_DIR}/Connector_PinHeader_2.54mm.3dshapes/PinHeader_1x03_P2.54mm_Vertical.wrl"
@@
   )
   (footprint "Resistor_SMD:R_0805_2012Metric_Pad1.20x1.40mm_HandSolder" (layer "B.Cu")
-    (at 136.9575 153.49 180)
+    (at 130.4775 145.26 180)
     (descr "Resistor SMD 0805 (2012 Metric), square (rectangular) end terminal, IPC_7351 nominal with elongated pad for handsoldering. (Body size source: IPC-SM-782 page 72, https://www.pcb-3d.com/wordpress/wp-content/uploads/ipc-sm-782a_amendment_1_and_2.pdf), generated with kicad-footprint-generator")
     (tags "resistor handsolder")
@@
   (segment (start 119.6475 135.63) (end 119.6475 138.56) (width 0.25) (layer "F.Cu") (net 3))
   (segment (start 108.3975 122.43) (end 109.6275 121.2) (width 0.25) (layer "B.Cu") (net 3))
+  (segment (start 143.8275 129.29) (end 134.7675 129.29) (width 0.25) (layer "B.Cu") (net 3))
+  (segment (start 145.8675 127.365) (end 145.7525 127.365) (width 0.25) (layer "B.Cu") (net 3))
   (segment (start 97.9925 111.5375) (end 97.9925 109.45) (width 0.25) (layer "B.Cu") (net 3))
   (segment (start 99.475 113.02) (end 97.9925 111.5375) (width 0.25) (layer "B.Cu") (net 3))
   (segment (start 131.5125 112.26) (end 129.0275 112.26) (width 0.25) (layer "B.Cu") (net 3))
   (segment (start 109.6275 121.2) (end 109.6275 118.8) (width 0.25) (layer "B.Cu") (net 3))
+  (segment (start 147.3575 118.015) (end 146.9325 117.59) (width 0.25) (layer "B.Cu") (net 3))
   (segment (start 146.9325 117.59) (end 146.0075 116.665) (width 0.25) (layer "B.Cu") (net 3))
   (segment (start 114.7075 144.36) (end 121.0075 144.36) (width 0.25) (layer "B.Cu") (net 3))
   (segment (start 100.2775 109.45) (end 97.9925 109.45) (width 0.25) (layer "B.Cu") (net 3))
-  (segment (start 146.9325 117.59) (end 147.2775 117.935) (width 0.25) (layer "B.Cu") (net 3))
+  (segment (start 145.8675 127.365) (end 147.3575 125.875) (width 0.25) (layer "B.Cu") (net 3))
+  (segment (start 145.7525 127.365) (end 143.8275 129.29) (width 0.25) (layer "B.Cu") (net 3))
   (segment (start 109.6275 118.8) (end 100.2775 109.45) (width 0.25) (layer "B.Cu") (net 3))
-  (segment (start 147.2775 117.935) (end 147.2775 127.685) (width 0.25) (layer "B.Cu") (net 3))
-  (segment (start 147.2775 127.685) (end 145.54 129.4225) (width 0.25) (layer "B.Cu") (net 3))
   (segment (start 132.0775 111.695) (end 131.5125 112.26) (width 0.25) (layer "B.Cu") (net 3))
   (segment (start 146.0075 116.665) (end 146.0075 112.215) (width 0.25) (layer "B.Cu") (net 3))
+  (segment (start 147.3575 125.875) (end 147.3575 118.015) (width 0.25) (layer "B.Cu") (net 3))
   (segment (start 123.25 141.0225) (end 124.88 139.3925) (width 0.25) (layer "F.Cu") (net 4))
   (segment (start 123.3375 144.96) (end 123.25 144.8725) (width 0.25) (layer "F.Cu") (net 4))
@@
   (segment (start 113.8475 145.8) (end 109.1875 145.8) (width 0.25) (layer "B.Cu") (net 4))
   (segment (start 130.7675 110.99) (end 129.0275 110.99) (width 0.25) (layer "B.Cu") (net 4))
+  (segment (start 135.6475 111.5975) (end 135.6475 109.92) (width 0.25) (layer "B.Cu") (net 4))
   (segment (start 136.3875 120.3) (end 136.735 119.9525) (width 0.25) (layer "B.Cu") (net 4))
   (segment (start 114.7075 146.66) (end 113.8475 145.8) (width 0.25) (layer "B.Cu") (net 4))
@@
   (segment (start 101.63 131.61) (end 101.63 127.935) (width 0.25) (layer "B.Cu") (net 4))
   (segment (start 135.6475 111.5975) (end 134.11 110.06) (width 0.25) (layer "B.Cu") (net 4))
+  (segment (start 138.4325 107.135) (end 146.0075 107.135) (width 0.25) (layer "B.Cu") (net 4))
   (segment (start 109.1875 142.15) (end 109.3175 142.02) (width 0.25) (layer "B.Cu") (net 4))
   (segment (start 109.1875 145.8) (end 109.1875 142.15) (width 0.25) (layer "B.Cu") (net 4))
   (segment (start 102.3275 127.1875) (end 101.605 127.91) (width 0.25) (layer "B.Cu") (net 4))
+  (segment (start 135.6475 109.92) (end 138.4325 107.135) (width 0.25) (layer "B.Cu") (net 4))
   (segment (start 126.8475 131.79) (end 126.2425 131.185) (width 0.25) (layer "B.Cu") (net 4))
   (segment (start 99.115 134.125) (end 101.63 131.61) (width 0.25) (layer "B.Cu") (net 4))
@@
   (segment (start 128.9075 135.27) (end 128.8875 135.25) (width 0.25) (layer "B.Cu") (net 21))
   (segment (start 131.5075 135.27) (end 128.9075 135.27) (width 0.25) (layer "B.Cu") (net 21))
-  (segment (start 123.9175 135.31) (end 123.8975 135.29) (width 0.25) (layer "B.Cu") (net 21))
   (segment (start 138.8275 122.52) (end 138.7275 122.42) (width 0.25) (layer "B.Cu") (net 23))
   (segment (start 138.8275 122.52) (end 138.7075 122.4) (width 0.25) (layer "B.Cu") (net 23))
@@
   (segment (start 100.8575 141.1) (end 100.8575 145.97) (width 0.25) (layer "B.Cu") (net 39))
   (segment (start 100.8575 145.97) (end 102.5875 147.7) (width 0.25) (layer "B.Cu") (net 39))
-  (segment (start 137.42 126.8825) (end 135.4975 124.96) (width 0.25) (layer "B.Cu") (net 62))
-  (segment (start 145.54 126.8825) (end 137.42 126.8825) (width 0.25) (layer "B.Cu") (net 62))
-  (segment (start 135.4975 124.96) (end 129.0275 124.96) (width 0.25) (layer "B.Cu") (net 62))
+  (segment (start 144.2225 124.825) (end 141.9675 127.08) (width 0.25) (layer "B.Cu") (net 62))
+  (segment (start 145.8675 124.825) (end 144.2225 124.825) (width 0.25) (layer "B.Cu") (net 62))
+  (segment (start 134.5975 124.96) (end 129.0275 124.96) (width 0.25) (layer "B.Cu") (net 62))
+  (segment (start 141.9675 127.08) (end 136.7175 127.08) (width 0.25) (layer "B.Cu") (net 62))
+  (segment (start 136.7175 127.08) (end 134.5975 124.96) (width 0.25) (layer "B.Cu") (net 62))
 )

Commit message: Update hardware.kicad_pcb
Parts:
- removed U107: DHT11, Sensor:Aosong_DHT11_5.5x12.0_P2.54mm
- moved D104 24.2 mm to (127.8, 146.8), turned to -90 degrees
- moved D106 20.7 mm to (140.4, 125.0), turned to 0 degrees
- moved J107 19.7 mm to (139.6, 153.4), turned to -90 degrees
- moved J105 18.4 mm to (127.8, 153.3), turned to 90 degrees
- moved R110 13.0 mm to (127.2, 139.5)
- moved R118 12.1 mm to (132.9, 147.1)
- moved R116 11.5 mm to (123.8, 135.9), turned to 90 degrees
- moved R112 4.39 mm to (135.4, 124.8)
- moved D103 0.97 mm to (133.8, 130.6)
Routing:
- net Net-(C113-Pad2): track 5.69 -> 30.5 mm, vias 0 -> 1
- net +3V3: track 78.2 -> 98.8 mm
- net GND: track 121.4 -> 130.4 mm
- net Net-(D104-Pad1): track 0.00 -> 6.45 mm
- net Net-(J105-Pad2): track 0.00 -> 6.30 mm
- net /LED4: track 10.3 -> 5.88 mm
- net /STDBY: track 0.00 -> 3.62 mm
- net /STDB: track 3.74 -> 6.98 mm
- net Net-(D106-Pad1): track 0.00 -> 3.01 mm
- net Net-(D103-Pad1): track 4.45 -> 3.80 mm
