File: hardware/hardware.kicad_pcb (KiCad board)
At the start: 2 copper layers, 55 parts, among them J101 VIN, J102 BAT, J103 DISPLAY, J104 EXT, J105 VIN, J106 SENSOR_DHT, J107 solo, SW101 BOOT, U101 LM324, U102 TP4056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

Commit message: Update hardware.kicad_pcb
Routing:
- net +3V3: track 98.8 -> 108.4 mm
Changed lines of the file:
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@@
   (segment (start 108.3975 122.43) (end 109.6275 121.2) (width 0.25) (layer "B.Cu") (net 3))
   (segment (start 121.0075 147.02) (end 121.0075 144.36) (width 0.25) (layer "B.Cu") (net 3))
+  (segment (start 141.4525 124.95) (end 142.5175 123.885) (width 0.25) (layer "B.Cu") (net 3))
+  (segment (start 142.5175 122.005) (end 146.9325 117.59) (width 0.25) (layer "B.Cu") (net 3))
   (segment (start 97.9925 111.5375) (end 97.9925 109.45) (width 0.25) (layer "B.Cu") (net 3))
   (segment (start 99.475 113.02) (end 97.9925 111.5375) (width 0.25) (layer "B.Cu") (net 3))
   (segment (start 131.5125 112.26) (end 129.0275 112.26) (width 0.25) (layer "B.Cu") (net 3))
   (segment (start 109.6275 121.2) (end 109.6275 118.8) (width 0.25) (layer "B.Cu") (net 3))
+  (segment (start 142.5175 123.885) (end 142.5175 122.005) (width 0.25) (layer "B.Cu") (net 3))
   (segment (start 127.7775 147.9) (end 127.7775 153.3) (width 0.25) (layer "B.Cu") (net 3))
   (segment (start 147.3575 118.015) (end 146.9325 117.59) (width 0.25) (layer "B.Cu") (net 3))

Commit message: Update hardware.kicad_pcb
Parts:
- moved C102 23.7 mm to (132.6, 141.7), turned to 0 degrees
Routing:
- net +3V3: track 108.4 -> 117.2 mm
- net GND: track 130.4 -> 135.1 mm
Changed lines of the file:
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@@
   )
   (footprint "Capacitor_SMD:C_0805_2012Metric_Pad1.18x1.45mm_HandSolder" (layer "B.Cu")
-    (at 156.2675 140.1325 -90)
+    (at 132.62 141.67)
     (descr "Capacitor SMD 0805 (2012 Metric), square (rectangular) end terminal, IPC_7351 nominal with elongated pad for handsoldering. (Body size source: IPC-SM-782 page 76, https://www.pcb-3d.com/wordpress/wp-content/uploads/ipc-sm-782a_amendment_1_and_2.pdf, https://docs.google.com/spreadsheets/d/1BsfQQcO9C6DZCsRaXUlFlo91Tg2WpOkGARC1WS5S8t0/edit?usp=sharing), generated with kicad-footprint-generator")
     (tags "capacitor handsolder")
@@
     (property "Sheetname" "")
     (attr smd)
-    (fp_text reference "C102" (at -0.4975 2.03 90) (layer "B.SilkS")
-      (effects (font (size 1 1) (thickness 0.15)) (justify mirror))
-    )
-    (fp_text value "100nF" (at -1.2375 1.44 90) (layer "B.Fab")
-      (effects (font (size 1 1) (thickness 0.15)) (justify mirror))
-    )
-    (fp_text user "${REFERENCE}" (at 0 0 90) (layer "B.Fab")
+    (fp_text reference "C102" (at -0.04 1.75) (layer "B.SilkS")
+      (effects (font (size 1 1) (thickness 0.15)) (justify mirror))
+    )
+    (fp_text value "100nF" (at -0.52 1.62) (layer "B.Fab")
+      (effects (font (size 1 1) (thickness 0.15)) (justify mirror))
+    )
+    (fp_text user "${REFERENCE}" (at 0 0) (layer "B.Fab")
       (effects (font (size 0.5 0.5) (thickness 0.08)) (justify mirror))
     )
@@
     (fp_line (start 1 -0.625) (end -1 -0.625) (layer "B.Fab") (width 0.1))
     (fp_line (start 1 0.625) (end 1 -0.625) (layer "B.Fab") (width 0.1))
-    (pad "1" smd roundrect (at -1.0375 0 270) (size 1.175 1.45) (layers "B.Cu" "B.Paste" "B.Mask") (roundrect_rratio 0.212766)
+    (pad "1" smd roundrect (at -1.0375 0) (size 1.175 1.45) (layers "B.Cu" "B.Paste" "B.Mask") (roundrect_rratio 0.212766)
       (net 3 "+3V3") (pintype "passive"))
-    (pad "2" smd roundrect (at 1.0375 0 270) (size 1.175 1.45) (layers "B.Cu" "B.Paste" "B.Mask") (roundrect_rratio 0.212766)
+    (pad "2" smd roundrect (at 1.0375 0) (size 1.175 1.45) (layers "B.Cu" "B.Paste" "B.Mask") (roundrect_rratio 0.212766)
       (net 4 "GND") (pintype "passive"))
     (model "${KICAD6_3DMODEL_DIR}/Capacitor_SMD.3dshapes/C_0805_2012Metric.wrl"
@@
   (segment (start 115.4075 153.3) (end 114.0375 151.93) (width 0.25) (layer "B.Cu") (net 3))
   (segment (start 108.3975 122.43) (end 109.6275 121.2) (width 0.25) (layer "B.Cu") (net 3))
+  (segment (start 130.3075 147.14) (end 129.5875 147.86) (width 0.25) (layer "B.Cu") (net 3))
   (segment (start 121.0075 147.02) (end 121.0075 144.36) (width 0.25) (layer "B.Cu") (net 3))
   (segment (start 141.4525 124.95) (end 142.5175 123.885) (width 0.25) (layer "B.Cu") (net 3))
@@
   (segment (start 97.9925 111.5375) (end 97.9925 109.45) (width 0.25) (layer "B.Cu") (net 3))
   (segment (start 99.475 113.02) (end 97.9925 111.5375) (width 0.25) (layer "B.Cu") (net 3))
+  (segment (start 130.3075 142.945) (end 130.3075 147.14) (width 0.25) (layer "B.Cu") (net 3))
   (segment (start 131.5125 112.26) (end 129.0275 112.26) (width 0.25) (layer "B.Cu") (net 3))
   (segment (start 109.6275 121.2) (end 109.6275 118.8) (width 0.25) (layer "B.Cu") (net 3))
@@
   (segment (start 145.8675 127.365) (end 147.3575 125.875) (width 0.25) (layer "B.Cu") (net 3))
   (segment (start 114.0375 151.93) (end 114.0375 150.1) (width 0.25) (layer "B.Cu") (net 3))
+  (segment (start 131.5825 141.67) (end 130.3075 142.945) (width 0.25) (layer "B.Cu") (net 3))
   (segment (start 127.8175 147.86) (end 127.7775 147.9) (width 0.25) (layer "B.Cu") (net 3))
   (segment (start 109.6275 118.8) (end 100.2775 109.45) (width 0.25) (layer "B.Cu") (net 3))
   (segment (start 115.2275 148.91) (end 119.1175 148.91) (width 0.25) (layer "B.Cu") (net 3))
+  (segment (start 129.5875 147.86) (end 127.8175 147.86) (width 0.25) (layer "B.Cu") (net 3))
   (segment (start 132.0775 111.695) (end 131.5125 112.26) (width 0.25) (layer "B.Cu") (net 3))
   (segment (start 127.7775 153.3) (end 115.4075 153.3) (width 0.25) (layer "B.Cu") (net 3))
@@
   (segment (start 100.3675 102.7) (end 100.3675 105.34) (width 0.25) (layer "B.Cu") (net 4))
   (segment (start 97.325 121.1275) (end 98.8975 121.1275) (width 0.25) (layer "B.Cu") (net 4))
+  (segment (start 132.8975 146.07) (end 132.8975 142.43) (width 0.25) (layer "B.Cu") (net 4))
   (segment (start 98.8975 121.1275) (end 99.225 121.1275) (width 0.25) (layer "B.Cu") (net 4))
   (segment (start 98.835 121.1275) (end 98.8975 121.1275) (width 0.25) (layer "B.Cu") (net 4))
@@
   (segment (start 113.8475 145.8) (end 109.1875 145.8) (width 0.25) (layer "B.Cu") (net 4))
   (segment (start 130.7675 110.99) (end 129.0275 110.99) (width 0.25) (layer "B.Cu") (net 4))
+  (segment (start 132.8975 142.43) (end 133.6575 141.67) (width 0.25) (layer "B.Cu") (net 4))
   (segment (start 137.0775 153.36) (end 137.0775 150.25) (width 0.25) (layer "B.Cu") (net 4))
   (segment (start 135.6475 111.5975) (end 135.6475 109.92) (width 0.25) (layer "B.Cu") (net 4))

Commit message: update pcb
Parts:
- moved R118 3.58 mm to (136.4, 146.5)
- moved C102 1.61 mm to (131.6, 142.9)
Routing:
- net Net-(J105-Pad2): track 6.30 -> 68.5 mm, vias 0 -> 1
- net GND: track 135.1 -> 126.1 mm
- net +3V3: track 117.2 -> 115.4 mm
- net /LUX_ADC: track 11.5 -> 13.2 mm
- net /SENS_SOLO: track 11.8 -> 12.5 mm

Commit message: Update hardware.kicad_pcb
Parts:
- moved D104 2.26 mm to (127.5, 144.6)
- moved C102 1.45 mm to (130.3, 142.5), turned to 90 degrees
Routing:
- net Net-(C113-Pad2): track 30.5 -> 90.4 mm
- net /CHRG: track 2.63 -> 55.4 mm, vias 0 -> 1
- net +3V3: track 115.4 -> 79.5 mm
- net GND: track 126.1 -> 121.4 mm
- net Net-(D104-Pad1): track 6.45 -> 4.34 mm
- net GND1: track 22.4 -> 20.6 mm
- net Net-(R119-Pad1): track 28.9 -> 30.1 mm

Commit message: update pcb
Parts:
- moved R107 1.51 mm to (106.9, 123.4)
Routing:
- net +3V3: track 79.5 -> 265.4 mm, vias 0 -> 4
- net /STDBY: track 3.62 -> 39.8 mm, vias 0 -> 1
- net GND: track 121.4 -> 100.4 mm
- net /CHRG: track 55.4 -> 57.6 mm
- net /IO0: track 12.5 -> 14.4 mm
- net Net-(J105-Pad2): track 68.5 -> 67.1 mm
- net Net-(D102-Pad2): track 46.7 -> 45.6 mm

Commit message: pcb
finalizado
- precisa revisar pcb e esquemático
Parts:
- added C120: 100nF, Capacitor_SMD:C_0805_2012Metric_Pad1.18x1.45mm_HandSolder, F.Cu at (103.5, 111.1)
- added J108: TX_RX, Connector_PinSocket_2.54mm:PinSocket_1x04_P2.54mm_Vertical, F.Cu at (98.5, 122.0)
- moved J107 17.2 mm to (146.0, 137.4), turned to 0 degrees
- moved J105 14.1 mm to (141.9, 153.4)
- moved D101 9.91 mm to (127.0, 153.8)
- moved D102 5.12 mm to (112.1, 154.0)
- moved R106 4.12 mm to (103.0, 132.0)
- moved C109 3.88 mm to (99.3, 116.2), turned to -90 degrees
- moved C106 2.91 mm to (103.0, 134.5)
- moved J101 2.80 mm to (98.1, 152.9), turned to 180 degrees
- moved J104 2.00 mm to (145.5, 110.3)
- moved C111 1.64 mm to (98.4, 111.4)
- moved J103 1.46 mm to (98.3, 108.0)
- moved R107 1.37 mm to (107.6, 124.5)
- moved R102 1.13 mm to (103.0, 141.7), turned to 90 degrees
- moved R104 1.10 mm to (132.1, 113.8)
- moved R103 0.93 mm to (111.6, 133.2), turned to 180 degrees
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Routing:
- net GND1: track 20.6 -> 89.9 mm, vias 0 -> 3
- net GND: track 100.4 -> 39.3 mm, vias 0 -> 14
- net /RX: track 0.00 -> 25.7 mm, vias 0 -> 2
- net +3V3: track 265.4 -> 291.0 mm
- net /TX: track 0.00 -> 25.5 mm, vias 0 -> 2
- net Net-(C113-Pad2): track 90.4 -> 71.8 mm
- net BAT+: track 64.6 -> 73.5 mm
- net Net-(J104-Pad2): track 74.8 -> 70.0 mm
- net Net-(D101-Pad1): track 34.0 -> 38.2 mm
- net /VBAT: track 29.9 -> 27.3 mm
- net Net-(U103-Pad3): track 17.4 -> 19.9 mm
- net Net-(J105-Pad2): track 67.1 -> 69.5 mm
- net /CHRG: track 57.6 -> 55.5 mm
- net /STDBY: track 39.8 -> 41.8 mm
- net Net-(R102-Pad2): track 4.81 -> 3.07 mm
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- added copper zone on B.Cu, net GND
- added copper zone on F.Cu, net GND
Other:
- board outline added: 53.5 x 59 mm

Commit message: update pcb
Other:
- board text added: "PI3 - 2022/1 Vaso Inteligente Guilherme Camargo Valese Ariane Andréia Martins"
Changed lines of the file:
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@@
   (gr_rect (start 95.5255 155.662) (end 148.0755 97.752) (layer "B.Cu") (width 0.2) (fill none))
   (gr_rect (start 95 97.238) (end 148.508 156.254) (layer "Edge.Cuts") (width 0.2) (fill none))
+  (gr_text "PI3 - 2022/1\nVaso Inteligente\nGuilherme Camargo Valese\nAriane Andréia Martins" (at 120.8575 102.8) (layer "F.Cu")
+    (effects (font (size 1 1) (thickness 0.15)))
+  )
   (segment (start 116.2275 147.8) (end 112.3615 151.666) (width 0.25) (layer "F.Cu") (net 1))
   (segment (start 108.7025 145.605) (end 110.2925 145.605) (width 0.25) (layer "F.Cu") (net 1))

Commit message: Update hardware.kicad_pcb
Routing:
- net GND: track 39.3 -> 46.6 mm, vias 14 -> 11
- net Net-(R119-Pad1): track 30.7 -> 32.7 mm
- net Net-(C113-Pad2): track 71.8 -> 71.1 mm
Changed lines of the file:
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@@
   (segment (start 123.3375 144.96) (end 123.25 144.8725) (width 0.25) (layer "F.Cu") (net 4))
   (segment (start 128.16 139.3925) (end 124.88 139.3925) (width 0.25) (layer "F.Cu") (net 4))
+  (segment (start 142.7875 106.04) (end 142.7275 105.98) (width 0.25) (layer "F.Cu") (net 4))
   (segment (start 128.1875 139.42) (end 128.16 139.3925) (width 0.25) (layer "F.Cu") (net 4))
-  (segment (start 142.5975 106.11) (end 142.7275 105.98) (width 0.25) (layer "F.Cu") (net 4))
-  (segment (start 142.5975 111.83) (end 142.5975 106.11) (width 0.25) (layer "F.Cu") (net 4))
   (segment (start 123.3375 148.59) (end 123.3375 144.96) (width 0.25) (layer "F.Cu") (net 4))
   (segment (start 123.25 144.8725) (end 123.25 141.0225) (width 0.25) (layer "F.Cu") (net 4))
-  (via (at 126.6675 114.53) (size 1) (drill 0.4) (layers "F.Cu" "B.Cu") (free) (net 4))
   (via (at 100.6375 113.62) (size 1) (drill 0.4) (layers "F.Cu" "B.Cu") (free) (net 4))
   (via (at 142.7275 105.98) (size 1) (drill 0.4) (layers "F.Cu" "B.Cu") (free) (net 4))
-  (via (at 116.6975 125.27) (size 1) (drill 0.4) (layers "F.Cu" "B.Cu") (free) (net 4))
   (via (at 138.6575 100.21) (size 1) (drill 0.4) (layers "F.Cu" "B.Cu") (free) (net 4))
   (via (at 141.4175 143.74) (size 1) (drill 0.4) (layers "F.Cu" "B.Cu") (free) (net 4))
   (via (at 143.2575 100.18) (size 1) (drill 0.4) (layers "F.Cu" "B.Cu") (free) (net 4))
-  (via (at 126.9675 123.99) (size 1) (drill 0.4) (layers "F.Cu" "B.Cu") (free) (net 4))
   (via (at 137.70449 118.14) (size 1) (drill 0.4) (layers "F.Cu" "B.Cu") (free) (net 4))
   (via (at 134.5975 149.27) (size 1) (drill 0.4) (layers "F.Cu" "B.Cu") (free) (net 4))
   (via (at 140.9175 100.21) (size 1) (drill 0.4) (layers "F.Cu" "B.Cu") (free) (net 4))
-  (via (at 118.5375 125.87) (size 1) (drill 0.4) (layers "F.Cu" "B.Cu") (free) (net 4))
-  (via (at 142.5975 111.83) (size 1) (drill 0.4) (layers "F.Cu" "B.Cu") (free) (net 4))
+  (via (at 142.7875 111.62) (size 1) (drill 0.4) (layers "F.Cu" "B.Cu") (free) (net 4))
+  (via (at 102.9975 102.76) (size 1) (drill 0.4) (layers "F.Cu" "B.Cu") (free) (net 4))
   (via (at 130.6475 139.39) (size 1) (drill 0.4) (layers "F.Cu" "B.Cu") (free) (net 4))
+  (segment (start 136.7225 111.06) (end 135.9275 111.855) (width 0.25) (layer "B.Cu") (net 4))
   (segment (start 142.7275 105.98) (end 143.5025 105.205) (width 0.25) (layer "B.Cu") (net 4))
   (segment (start 126.2425 131.185) (end 126.2425 128.5) (width 0.25) (layer "B.Cu") (net 4))
   (segment (start 98.5975 134.125) (end 99.115 134.125) (width 0.25) (layer "B.Cu") (net 4))
   (segment (start 136.0475 117.445) (end 135.9925 117.39) (width 0.25) (layer "B.Cu") (net 4))
-  (segment (start 142.5975 111.83) (end 141.8275 111.06) (width 0.25) (layer "B.Cu") (net 4))
+  (segment (start 142.7875 111.62) (end 142.2275 111.06) (width 0.25) (layer "B.Cu") (net 4))
+  (segment (start 142.2275 111.06) (end 136.7225 111.06) (width 0.25) (layer "B.Cu") (net 4))
   (segment (start 136.0475 120.1) (end 136.0475 117.445) (width 0.25) (layer "B.Cu") (net 4))
   (segment (start 118.6675 131.69) (end 121.6475 131.69) (width 0.25) (layer "B.Cu") (net 4))
-  (segment (start 136.7225 111.06) (end 135.9275 111.855) (width 0.25) (layer "B.Cu") (net 4))
-  (segment (start 141.8275 111.06) (end 136.7225 111.06) (width 0.25) (layer "B.Cu") (net 4))
+  (segment (start 121.5275 114.38) (end 124.9175 110.99) (width 0.25) (layer "B.Cu") (net 4))
+  (segment (start 124.9175 110.99) (end 129.0275 110.99) (width 0.25) (layer "B.Cu") (net 4))
+  (segment (start 121.5275 118.49) (end 121.5275 114.38) (width 0.25) (layer "B.Cu") (net 4))
   (segment (start 143.5025 105.205) (end 145.4675 105.205) (width 0.25) (layer "B.Cu") (net 4))
   (segment (start 126.8475 131.79) (end 126.2425 131.185) (width 0.25) (layer "B.Cu") (net 4))
@@
   (segment (start 138.1075 113.47) (end 138.1075 114.66) (width 0.25) (layer "B.Cu") (net 25))
   (segment (start 133.8675 117.34) (end 129.0275 117.34) (width 0.25) (layer "B.Cu") (net 25))
+  (segment (start 137.7575 114.58) (end 132.6575 119.68) (width 0.25) (layer "F.Cu") (net 26))
+  (segment (start 145.2875 118.47) (end 145.2875 116.04) (width 0.25) (layer "F.Cu") (net 26))
+  (segment (start 143.8275 114.58) (end 137.7575 114.58) (width 0.25) (layer "F.Cu") (net 26))
+  (segment (start 145.2875 116.04) (end 143.8275 114.58) (width 0.25) (layer "F.Cu") (net 26))
   (segment (start 132.6575 119.68) (end 126.714251 119.68) (width 0.25) (layer "F.Cu") (net 26))
-  (segment (start 126.714251 119.68) (end 125.244251 118.21) (width 0.25) (layer "F.Cu") (net 26))
-  (segment (start 145.2875 118.47) (end 145.2875 114.84) (width 0.25) (layer "F.Cu") (net 26))
   (segment (start 142.9775 137.37) (end 135.1175 137.37) (width 0.25) (layer "F.Cu") (net 26))
-  (segment (start 125.244251 118.21) (end 124.8675 118.21) (width 0.25) (layer "F.Cu") (net 26))
   (segment (start 135.0925 137.345) (end 128.1875 137.345) (width 0.25) (layer "F.Cu") (net 26))
-  (segment (start 142.9775 137.37) (end 141.1075 135.5) (width 0.25) (layer "F.Cu") (net 26))
   (segment (start 124.1275 134.84) (end 126.6975 134.84) (width 0.25) (layer "F.Cu") (net 26))
   (segment (start 126.6975 134.84) (end 128.1875 136.33) (width 0.25) (layer "F.Cu") (net 26))
   (segment (start 135.1175 137.37) (end 135.0925 137.345) (width 0.25) (layer "F.Cu") (net 26))
-  (segment (start 145.0275 114.58) (end 137.7575 114.58) (width 0.25) (layer "F.Cu") (net 26))
+  (segment (start 141.1075 135.5) (end 141.1075 122.65) (width 0.25) (layer "F.Cu") (net 26))
+  (segment (start 125.244251 118.21) (end 124.8675 118.21) (width 0.25) (layer "F.Cu") (net 26))
+  (segment (start 128.1875 136.33) (end 128.1875 137.345) (width 0.25) (layer "F.Cu") (net 26))
+  (segment (start 126.714251 119.68) (end 125.244251 118.21) (width 0.25) (layer "F.Cu") (net 26))
+  (segment (start 142.9775 137.37) (end 141.1075 135.5) (width 0.25) (layer "F.Cu") (net 26))
   (segment (start 141.1075 122.65) (end 145.2875 118.47) (width 0.25) (layer "F.Cu") (net 26))
-  (segment (start 137.7575 114.58) (end 132.6575 119.68) (width 0.25) (layer "F.Cu") (net 26))
-  (segment (start 128.1875 136.33) (end 128.1875 137.345) (width 0.25) (layer "F.Cu") (net 26))
-  (segment (start 141.1075 135.5) (end 141.1075 122.65) (width 0.25) (layer "F.Cu") (net 26))
-  (segment (start 145.2875 114.84) (end 145.0275 114.58) (width 0.25) (layer "F.Cu") (net 26))
   (via (at 142.9775 137.37) (size 1) (drill 0.4) (layers "F.Cu" "B.Cu") (net 26))
   (segment (start 142.9925 137.355) (end 142.9775 137.37) (width 0.25) (layer "B.Cu") (net 26))
@@
   (segment (start 123.7875 131.83) (end 123.6475 131.69) (width 0.25) (layer "B.Cu") (net 30))
   (segment (start 123.7875 134.87) (end 123.7875 131.83) (width 0.25) (layer "B.Cu") (net 30))
-  (segment (start 122.5575 113.03) (end 119.9175 115.67) (width 0.25) (layer "F.Cu") (net 31))
-  (segment (start 143.6175 113.58) (end 143.0675 113.03) (width 0.25) (layer "F.Cu") (net 31))
-  (segment (start 143.0675 113.03) (end 122.5575 113.03) (width 0.25) (layer "F.Cu") (net 31))
+  (segment (start 122.9375 112.65) (end 119.9175 115.67) (width 0.25) (layer "F.Cu") (net 31))
+  (segment (start 144.0575 112.65) (end 122.9375 112.65) (width 0.25) (layer "F.Cu") (net 31))
+  (segment (start 144.3475 112.36) (end 144.0575 112.65) (width 0.25) (layer "F.Cu") (net 31))
   (segment (start 119.9175 116.94) (end 119.9175 115.67) (width 0.25) (layer "F.Cu") (net 31))
-  (via (at 143.6175 113.58) (size 1) (drill 0.4) (layers "F.Cu" "B.Cu") (free) (net 31))
-  (segment (start 143.6175 113.58) (end 142.7375 114.46) (width 0.25) (layer "B.Cu") (net 31))
-  (segment (start 142.7375 114.46) (end 139.6175 114.46) (width 0.25) (layer "B.Cu") (net 31))
+  (via (at 144.3475 112.36) (size 1) (drill 0.4) (layers "F.Cu" "B.Cu") (free) (net 31))
+  (segment (start 142.2475 114.46) (end 139.6175 114.46) (width 0.25) (layer "B.Cu") (net 31))
+  (segment (start 144.3475 112.36) (end 142.2475 114.46) (width 0.25) (layer "B.Cu") (net 31))
   (segment (start 119.9175 123.29) (end 119.9175 122.02) (width 0.25) (layer "F.Cu") (net 32))
   (segment (start 119.9175 123.47) (end 119.9175 123.29) (width 0.25) (layer "F.Cu") (net 32))
+  (segment (start 132.4575 125.62) (end 122.0675 125.62) (width 0.25) (layer "F.Cu") (net 32))
+  (segment (start 142.5975 117.24) (end 140.8375 117.24) (width 0.25) (layer "F.Cu") (net 32))
+  (segment (start 140.8375 117.24) (end 132.4575 125.62) (width 0.25) (layer "F.Cu") (net 32))
   (segment (start 122.0675 125.62) (end 119.9175 123.47) (width 0.25) (layer "F.Cu") (net 32))
-  (segment (start 131.9675 125.62) (end 122.0675 125.62) (width 0.25) (layer "F.Cu") (net 32))
-  (segment (start 140.3475 117.24) (end 131.9675 125.62) (width 0.25) (layer "F.Cu") (net 32))
-  (segment (start 142.5975 117.24) (end 140.3475 117.24) (width 0.25) (layer "F.Cu") (net 32))
   (via (at 142.5975 117.24) (size 1) (drill 0.4) (layers "F.Cu" "B.Cu") (free) (net 32))
   (segment (start 140.3975 117.24) (end 139.5675 116.41) (width 0.25) (layer "B.Cu") (net 32))
