File: hardware/hardware.kicad_pcb (KiCad board)
At the start: 2 copper layers, 53.5 x 59 mm, 57 parts, among them J101 VIN, J102 BAT, J103 DISPLAY, J104 EXT, J105 VIN, J106 SENSOR_DHT, J107 solo, J108 TX_RX, SW101 BOOT, U101 LM324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

Commit message: update pcb
Routing:
- net GND: track 46.6 -> 33.6 mm
Changed lines of the file:
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@@
   (segment (start 136.0475 120.1) (end 136.0475 117.445) (width 0.25) (layer "B.Cu") (net 4))
   (segment (start 118.6675 131.69) (end 121.6475 131.69) (width 0.25) (layer "B.Cu") (net 4))
-  (segment (start 121.5275 114.38) (end 124.9175 110.99) (width 0.25) (layer "B.Cu") (net 4))
-  (segment (start 124.9175 110.99) (end 129.0275 110.99) (width 0.25) (layer "B.Cu") (net 4))
-  (segment (start 121.5275 118.49) (end 121.5275 114.38) (width 0.25) (layer "B.Cu") (net 4))
   (segment (start 143.5025 105.205) (end 145.4675 105.205) (width 0.25) (layer "B.Cu") (net 4))
   (segment (start 126.8475 131.79) (end 126.2425 131.185) (width 0.25) (layer "B.Cu") (net 4))

Commit message: atualizado codigo
Parts:
- moved C107 75.7 mm to (52.5, 111.0)
- moved C112 75.7 mm to (64.8, 89.0)
- moved R111 75.7 mm to (69.0, 94.7)
- moved R121 75.7 mm to (64.8, 91.7)
- moved C101 75.7 mm to (43.5, 112.8)
- moved C103 75.7 mm to (35.9, 113.1)
- moved C105 75.7 mm to (65.7, 84.5)
- moved C108 75.7 mm to (52.0, 116.5)
- moved C111 75.7 mm to (28.2, 83.0)
- moved C120 75.7 mm to (33.3, 82.7)
- moved D101 75.7 mm to (56.8, 125.3)
- moved D103 75.7 mm to (63.6, 102.2)
- moved D104 75.7 mm to (57.3, 116.2)
- moved D105 75.7 mm to (75.7, 89.2)
- moved D106 75.7 mm to (70.3, 97.3)
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Connections:
- U102 pad 9: unconnected-(U102-Pad9) -> Net-(C101-Pad1)
Routing:
- net GND1: track 89.9 -> 70.6 mm, vias 3 -> 4
- net +3V3: track 290.6 -> 285.7 mm
- net Net-(C113-Pad2): track 71.1 -> 68.0 mm
- net /CHRG: track 55.5 -> 57.7 mm
- net Net-(C101-Pad1): track 44.4 -> 42.9 mm
- net Net-(J105-Pad2): track 69.5 -> 68.1 mm
- net Net-(D105-Pad1): track 8.24 -> 7.47 mm
- net /RX: track 25.7 -> 25.1 mm
- net Net-(D103-Pad1): track 3.80 -> 4.33 mm
- net Net-(J104-Pad2): track 70.0 -> 70.5 mm
- net GND: track 33.6 -> 33.1 mm, vias 11 -> 12

Commit message: adicionado função do luximetro
Routing:
- net Net-(D101-Pad1): track 38.2 -> 39.2 mm
- net /TX: track 25.9 -> 25.3 mm
