File: hardware/hardware.kicad_sch (KiCad schematic)
At the start: 45 parts, among them J101 VIN, J102 BAT, J103 DISPLAY, SW101 BOOT, U101 LM324, U102 TP4056, U103 DW01, U104 FS8205A, U105 AMS1117-3.3, U106 ESP32-WROOM-32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

Commit message: atualizado esquemático
Parts:
- removed U107: DHT11, Sensor:Aosong_DHT11_5.5x12.0_P2.54mm, symbol Sensor:DHT11
- added C112, C113: 100nF, Capacitor_SMD:C_0805_2012Metric_Pad1.18x1.45mm_HandSolder, symbol Device:C_Small
- added J104: EXT, Connector_PinHeader_2.54mm:PinHeader_1x03_P2.54mm_Vertical, symbol Connector:Conn_01x03_Male
- added J105: VIN, Connector_PinHeader_2.54mm:PinHeader_1x02_P2.54mm_Vertical, symbol Connector_Generic:Conn_01x02
- added J106: SENSOR_DHT, Connector_PinHeader_2.54mm:PinHeader_1x03_P2.54mm_Vertical, symbol Connector:Conn_01x03_Male
- added J107: solo, Connector_PinHeader_2.54mm:PinHeader_1x02_P2.54mm_Vertical, symbol Connector:Conn_01x02_Male
- added R118, R119, R122: 12K, Resistor_SMD:R_0805_2012Metric_Pad1.20x1.40mm_HandSolder, symbol Device:R_Small
- added R120: OPEN, Resistor_SMD:R_0805_2012Metric_Pad1.20x1.40mm_HandSolder, symbol Device:R_Small
- added R121: 0R, Resistor_SMD:R_0805_2012Metric_Pad1.20x1.40mm_HandSolder, symbol Device:R_Small
Connections:
- net +3V3: now also J104.1 (Pin_1), J105.1 (Pin_1), J106.1 (Pin_1), R122.1
- net DHT: now also U106.12 (IO27), J106.2 (Pin_2)
- net GND: now also C112.1, C113.1, J104.3 (Pin_3), J106.3 (Pin_3), J107.2 (Pin_2), R118.2, R121.1
- net LED4: now also U106.11 (IO26)
- net LUMINOSIDADE: now also U101.9 (-)
- net SENS_SOLO: now also U106.7 (IO35)
- net ST: now also U106.10 (IO25)
- net VBAT: now also U101.3 (+)
- net CHG: now reaches R114.2, R115.1
- net CHG: now also U106.13 (IO14)
- net at U101.10 (+): now also J105.2 (Pin_2), R118.1
- net STDB: now reaches R116.2, R117.1
- net STDB: now also U106.16 (IO13)
- net at U101.12 (+): now also C113.2, J107.1 (Pin_1), R122.2
- net IN1: now reaches U106.23 (IO15)
- net IN2: now reaches U106.26 (IO4)
- net VBAT_ADC: now reaches U106.6 (IO34)
- net VBAT_ADC: now also C112.2, R119.2
- net ADC_EXT: now reaches U106.8 (IO32)
- net ADC_EXT: now also R120.2, R121.2
- net LUX_ADC: now reaches U106.9 (IO33)
- net at U101.5 (+): now also J104.2 (Pin_2)
- net at U101.6 (-): now also U101.7, R120.1
- net at U101.1: now also U101.2 (-), R119.1
Other:
- note added: "Carregador de Bateria"
- note added: "Entradas Analógicas"
- note removed: "Alimentação"
- moved on the sheet: C102, C105, C110, C111, J103, R104, R107, R108, U101A, U101B, U101C, U101D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

Commit message: esq e pcb
Connections:
- net SCL: now also U106.36 (IO22)
- net SDA: now also U106.33 (IO21)
Changed lines of the file:
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@@
+    (stroke (width 0) (type default) (color 0 0 0 0))
+  )
+  (wire (pts (xy 148.59 154.94) (xy 156.21 154.94))
     (stroke (width 0) (type default) (color 0 0 0 0))
   )
@@
   )
   (wire (pts (xy 68.58 163.83) (xy 48.26 163.83))
+    (stroke (width 0) (type default) (color 0 0 0 0))
+  )
+  (wire (pts (xy 156.21 152.4) (xy 148.59 152.4))
     (stroke (width 0) (type default) (color 0 0 0 0))
   )
@@
     (effects (font (size 1.27 1.27)) (justify left bottom))
   )
+  (label "SDA" (at 156.21 152.4 0)
+    (effects (font (size 1.27 1.27)) (justify left bottom))
+  )
   (label "SENS_SOLO" (at 162.56 175.26 180)
     (effects (font (size 1.27 1.27)) (justify right bottom))
@@
     (effects (font (size 1.27 1.27)) (justify left bottom))
   )
+  (label "SCL" (at 156.21 154.94 0)
+    (effects (font (size 1.27 1.27)) (justify left bottom))
+  )

Commit message: update sch
Connections:
- net LUMINOSIDADE is gone; now on net LUX_ADC: U101.8, U101.9 (-)
Changed lines of the file:
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@@
     (effects (font (size 1.27 1.27)) (justify right bottom))
   )
-  (label "LUMINOSIDADE" (at 83.82 156.21 180)
+  (label "LUX_ADC" (at 83.82 156.21 180)
     (effects (font (size 1.27 1.27)) (justify right bottom))
   )
