File: hardware/hardware.kicad_sch (KiCad schematic)
At the start: 57 parts, among them J101 VIN, J102 BAT, J103 DISPLAY, J104 EXT, J105 VIN, J106 SENSOR_DHT, J107 solo, J108 TX_RX, SW101 BOOT, U101 LM324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

Commit message: atualizado pcb
Parts:
- removed C101, C103, C107: 10uF, Capacitor_SMD:CP_Elec_5x3, symbol Device:C_Polarized_Small
- removed C102, C104, C105, C106, C108, C110, C111, C112, C113, C120: 100nF, Capacitor_SMD:C_0805_2012Metric_Pad1.18x1.45mm_HandSolder, symbol Device:C_Small
- removed C109: 1nF, Capacitor_SMD:C_0805_2012Metric_Pad1.18x1.45mm_HandSolder, symbol Device:C_Small
- removed D101, D102: M7, Diode_SMD:D_MiniMELF_Handsoldering, symbol Device:D_Small
- removed D103: LED1, LED_SMD:LED_0805_2012Metric_Pad1.15x1.40mm_HandSolder, symbol Device:LED_Small
- removed D104: LED2, LED_SMD:LED_0805_2012Metric_Pad1.15x1.40mm_HandSolder, symbol Device:LED_Small
- removed D105: LED3, LED_SMD:LED_0805_2012Metric_Pad1.15x1.40mm_HandSolder, symbol Device:LED_Small
- removed D106: LED4, LED_SMD:LED_0805_2012Metric_Pad1.15x1.40mm_HandSolder, symbol Device:LED_Small
- removed J101, J105: VIN, Connector_PinHeader_2.54mm:PinHeader_1x02_P2.54mm_Vertical, symbol Connector_Generic:Conn_01x02
- removed J102: BAT, Connector_PinHeader_2.54mm:PinHeader_1x02_P2.54mm_Vertical, symbol Connector_Generic:Conn_01x02
- removed J103: DISPLAY, Connector_PinSocket_2.54mm:PinSocket_1x04_P2.54mm_Vertical, symbol Connector:Conn_01x04_Female
- removed J104: EXT, Connector_PinHeader_2.54mm:PinHeader_1x03_P2.54mm_Vertical, symbol Connector:Conn_01x03_Male
- removed J106: SENSOR_DHT, Connector_PinHeader_2.54mm:PinHeader_1x03_P2.54mm_Vertical, symbol Connector:Conn_01x03_Male
- removed J107: solo, Connector_PinHeader_2.54mm:PinHeader_1x02_P2.54mm_Vertical, symbol Connector:Conn_01x02_Male
- removed J108: TX_RX, Connector_PinSocket_2.54mm:PinSocket_1x04_P2.54mm_Vertical, symbol Connector:Conn_01x04_Female
- removed R101: 10k, Resistor_SMD:R_0805_2012Metric_Pad1.20x1.40mm_HandSolder, symbol Device:R
- removed R102: 1k, Resistor_SMD:R_0805_2012Metric_Pad1.20x1.40mm_HandSolder, symbol Device:R
- removed R103: 100, Resistor_SMD:R_0805_2012Metric_Pad1.20x1.40mm_HandSolder, symbol Device:R
- removed R104, R118, R119, R122: 12K, Resistor_SMD:R_0805_2012Metric_Pad1.20x1.40mm_HandSolder, symbol Device:R_Small
- removed R105, R106, R109, R110, R111, R112, R114, R115, R116, R117: R, Resistor_SMD:R_0805_2012Metric_Pad1.20x1.40mm_HandSolder, symbol Device:R_Small
- removed R107, R108: 4k7, Resistor_SMD:R_0805_2012Metric_Pad1.20x1.40mm_HandSolder, symbol Device:R_Small
- removed R113: 470, Resistor_SMD:R_0805_2012Metric_Pad1.20x1.40mm_HandSolder, symbol Device:R_Small
- removed R120: OPEN, Resistor_SMD:R_0805_2012Metric_Pad1.20x1.40mm_HandSolder, symbol Device:R_Small
- removed R121: 0R, Resistor_SMD:R_0805_2012Metric_Pad1.20x1.40mm_HandSolder, symbol Device:R_Small
- removed SW101: BOOT, Button_Switch_SMD:SW_SPST_CK_RS282G05A3, symbol Switch:SW_Push
- removed U101: LM324, Package_SO:SOIC-14_3.9x8.7mm_P1.27mm, symbol Amplifier_Operational:LM324
- removed U102: TP4056, Package_SO:SOIC-8-1EP_3.9x4.9mm_P1.27mm_EP2.29x3mm, symbol tp4056:TP4056
- removed U103: DW01, Package_TO_SOT_SMD:SOT-23-6_Handsoldering, symbol dw01:DW01
- removed U104: FS8205A, Package_TO_SOT_SMD:SOT-23-6_Handsoldering, symbol fs8205:FS8205A
- removed U105: AMS1117-3.3, Package_TO_SOT_SMD:SOT-223-3_TabPin2, symbol Regulator_Linear:AMS1117-3.3
- removed U106: ESP32-WROOM-32, RF_Module:ESP32-WROOM-32, symbol RF_Module:ESP32-WROOM-32
- added D? (x2): LED_Small, LED_SMD:LED_0805_2012Metric_Pad1.15x1.40mm_HandSolder, symbol Device:LED_Small
- added D?: (no value), symbol Device:LED_Small
- added R? (x2): R_Small, Resistor_SMD:R_0805_2012Metric_Pad1.20x1.40mm_HandSolder, symbol Device:R_Small
- added R?: (no value), symbol Device:R_Small
- added U?: (no value), symbol Memory_Flash:GD25D10CT
- added U?: (no value), symbol MCU_Espressif:ESP8266EX
- added Y?: (no value), symbol Device:Crystal
Connections:
- net GND: now also U?.33 (GND)
- new net: U?.28 (XTAL_IN), Y?.1
- new net: U?.27 (XTAL_OUT), Y?.2
- no-connect marks 3 -> 0
Other:
- note removed: "Carregador de Bateria"
- note removed: "Entradas Analógicas"
- company: PI3 - 2022/1 -> (none)
- title: Vaso Inteligente -> (none)
